File: PCB-Condenser-Microphone/PCB-Condenser-Microphone.sch (KiCad schematic (older format))
At the start: 2 parts

Commit message: Created schimatic and added digikey BOM
Parts:
- removed U?: SJ-3523-SMT, symbol Audio-Jack:SJ-3523-SMT
- added C1: 0.47uF, symbol device:C
- added C2, C3, C4: 10uF, symbol device:C
- added D1: LED, symbol device:LED
- added J1: Conn_01x02, symbol Connector:Conn_01x02
- added J2: SJ-3523-SMT, symbol Audio-Jack:SJ-3523-SMT
- added R1, R2: 1k, symbol device:R
- added R3, R4, R5, R6, R7: 10k, symbol device:R
- added R8: 100k, symbol device:R
- added RV1: 100k, symbol device:POT
- added SW1: SW_SPDT, symbol Switch:SW_SPDT
- added U1: LM358, symbol linear:LM358
- gave numbers to parts that had none: 1
Connections:
- net labels added: +9V
- wire segments 3 -> 48

Commit message: Added Titles
Parts:
- added MT1, MT2: Strain Relief, Mounting_Holes:MountingHole_2.2mm_M2, symbol Mechanical:Mounting_Hole
- C1: footprint (none) -> Capacitors_SMD:C_0603_HandSoldering
- C2, C3, C4: footprint (none) -> Capacitors_SMD:C_0805_HandSoldering
- D1: footprint (none) -> LEDs:LED_0603_HandSoldering
- J1: footprint (none) -> Pin_Headers:Pin_Header_Angled_1x02_Pitch2.54mm
- J2: footprint (none) -> PCB-Condenser-Microphone:SJ-3523-SMT-TR
- MK1: footprint (none) -> PCB-Condenser-Microphone:Condenser-Microphone-Backplate-30mm-Single-mount
- R1, R2, R3, R4, R5, R6, R7, R8: footprint (none) -> Resistors_SMD:R_0402
- RV1: footprint (none) -> PCB-Condenser-Microphone:TC33X
- SW1: footprint (none) -> Buttons_Switches_SMD:SW_SPDT_CK-JS102011SAQN
- U1: footprint (none) -> Housings_SOIC:SOIC-8_3.9x4.9mm_Pitch1.27mm
Changed lines of the file:
@@
 encoding utf-8
 Sheet 1 1
-Title ""
-Date ""
-Rev ""
+Title "PCB Condenser Microphone"
+Date "2018-03-13"
+Rev "1"
 Comp ""
 Comment1 ""
@@
 F 0 "MK1" H 2330 4846 50  0000 L CNN
 F 1 "Microphone_Condenser" H 2330 4755 50  0000 L CNN
-F 2 "" V 2200 4900 50  0001 C CNN
+F 2 "PCB-Condenser-Microphone:Condenser-Microphone-Backplate-30mm-Single-mount" V 2200 4900 50  0001 C CNN
 F 3 "" V 2200 4900 50  0001 C CNN
 	1    2200 4800
@@
 L Connector:Conn_01x02 J1
 U 1 1 5AA797B8
-P 1050 1500
-F 0 "J1" H 1200 1200 50  0000 C CNN
-F 1 "Conn_01x02" H 1200 1300 50  0000 C CNN
-F 2 "" H 1050 1500 50  0001 C CNN
-F 3 "~" H 1050 1500 50  0001 C CNN
-	1    1050 1500
+P 1750 1500
+F 0 "J1" H 1900 1200 50  0000 C CNN
+F 1 "Conn_01x02" H 1900 1300 50  0000 C CNN
+F 2 "Pin_Headers:Pin_Header_Angled_1x02_Pitch2.54mm" H 1750 1500 50  0001 C CNN
+F 3 "~" H 1750 1500 50  0001 C CNN
+	1    1750 1500
 	-1   0    0    1
 $EndComp
@@
 L power:GND #PWR0103
 U 1 1 5AA79854
-P 1900 1600
-F 0 "#PWR0103" H 1900 1350 50  0001 C CNN
-F 1 "GND" H 1905 1427 50  0000 C CNN
-F 2 "" H 1900 1600 50  0001 C CNN
-F 3 "" H 1900 1600 50  0001 C CNN
-	1    1900 1600
+P 2600 1600
+F 0 "#PWR0103" H 2600 1350 50  0001 C CNN
+F 1 "GND" H 2605 1427 50  0000 C CNN
+F 2 "" H 2600 1600 50  0001 C CNN
+F 3 "" H 2600 1600 50  0001 C CNN
+	1    2600 1600
 	1    0    0    -1
 $EndComp
@@
 L power:+9V #PWR0104
 U 1 1 5AA798F1
-P 1900 1300
-F 0 "#PWR0104" H 1900 1150 50  0001 C CNN
-F 1 "+9V" H 1915 1473 50  0000 C CNN
-F 2 "" H 1900 1300 50  0001 C CNN
-F 3 "" H 1900 1300 50  0001 C CNN
-	1    1900 1300
+P 2600 1300
+F 0 "#PWR0104" H 2600 1150 50  0001 C CNN
+F 1 "+9V" H 2615 1473 50  0000 C CNN
+F 2 "" H 2600 1300 50  0001 C CNN
+F 3 "" H 2600 1300 50  0001 C CNN
+	1    2600 1300
 	1    0    0    -1
 $EndComp
@@
 F 0 "R3" H 2270 4196 50  0000 L CNN
 F 1 "10k" H 2270 4105 50  0000 L CNN
-F 2 "" V 2130 4150 50  0001 C CNN
+F 2 "Resistors_SMD:R_0402" V 2130 4150 50  0001 C CNN
 F 3 "" H 2200 4150 50  0001 C CNN
 	1    2200 4150
@@
 F 0 "C3" V 2498 4450 50  0000 C CNN
 F 1 "10uF" V 2589 4450 50  0000 C CNN
-F 2 "" H 2788 4300 50  0001 C CNN
+F 2 "Capacitors_SMD:C_0805_HandSoldering" H 2788 4300 50  0001 C CNN
 F 3 "" H 2750 4450 50  0001 C CNN
 	1    2750 4450
@@
 F 0 "C4" V 7698 4100 50  0000 C CNN
 F 1 "10uF" V 7789 4100 50  0000 C CNN
-F 2 "" H 7988 3950 50  0001 C CNN
+F 2 "Capacitors_SMD:C_0805_HandSoldering" H 7988 3950 50  0001 C CNN
 F 3 "" H 7950 4100 50  0001 C CNN
 	1    7950 4100
@@
 L device:C C2
 U 1 1 5AA7A941
-P 2150 1450
-F 0 "C2" H 2035 1404 50  0000 R CNN
-F 1 "10uF" H 2035 1495 50  0000 R CNN
-F 2 "" H 2188 1300 50  0001 C CNN
-F 3 "" H 2150 1450 50  0001 C CNN
-	1    2150 1450
+P 2850 1450
+F 0 "C2" H 2735 1404 50  0000 R CNN
+F 1 "10uF" H 2735 1495 50  0000 R CNN
+F 2 "Capacitors_SMD:C_0805_HandSoldering" H 2888 1300 50  0001 C CNN
+F 3 "" H 2850 1450 50  0001 C CNN
+	1    2850 1450
 	-1   0    0    1
 $EndComp
 Wire Wire Line
-	1900 1300 2150 1300
-Wire Wire Line
-	1900 1600 2150 1600
+	2600 1300 2850 1300
+Wire Wire Line
+	2600 1600 2850 1600
 $Comp
 L device:LED D1
@@
 F 0 "D1" V 3738 1783 50  0000 R CNN
 F 1 "LED" V 3647 1783 50  0000 R CNN
-F 2 "" H 3700 1900 50  0001 C CNN
+F 2 "LEDs:LED_0603_HandSoldering" H 3700 1900 50  0001 C CNN
 F 3 "~" H 3700 1900 50  0001 C CNN
 	1    3700 1900
@@
 F 0 "R1" H 3770 2346 50  0000 L CNN
 F 1 "1k" H 3770 2255 50  0000 L CNN
-F 2 "" V 3630 2300 50  0001 C CNN
+F 2 "Resistors_SMD:R_0402" V 3630 2300 50  0001 C CNN
 F 3 "" H 3700 2300 50  0001 C CNN
 	1    3700 2300
@@
 L Switch:SW_SPDT SW1
 U 1 1 5AA7B7C5
-P 1550 1400
-F 0 "SW1" H 1550 1685 50  0000 C CNN
-F 1 "SW_SPDT" H 1550 1594 50  0000 C CNN
-F 2 "" H 1550 1400 50  0001 C CNN
-F 3 "" H 1550 1400 50  0001 C CNN
-	1    1550 1400
-	1    0    0    -1
-$EndComp
-Wire Wire Line
-	1250 1400 1350 1400
-Wire Wire Line
-	1750 1300 1900 1300
-Connection ~ 1900 1300
-Wire Wire Line
-	1250 1500 1250 1600
-Wire Wire Line
-	1250 1600 1900 1600
-Connection ~ 1900 1600
+P 2250 1400
+F 0 "SW1" H 2250 1685 50  0000 C CNN
+F 1 "SW_SPDT" H 2250 1594 50  0000 C CNN
+F 2 "Buttons_Switches_SMD:SW_SPDT_CK-JS102011SAQN" H 2250 1400 50  0001 C CNN
+F 3 "" H 2250 1400 50  0001 C CNN
+	1    2250 1400
+	1    0    0    -1
+$EndComp
+Wire Wire Line
+	1950 1400 2050 1400
+Wire Wire Line
+	2450 1300 2600 1300
+Connection ~ 2600 1300
+Wire Wire Line
+	1950 1500 1950 1600
+Wire Wire Line
+	1950 1600 2600 1600
+Connection ~ 2600 1600
 $Comp
 L linear:LM358 U1
@@
 F 0 "U1" H 4691 4396 50  0000 L CNN
 F 1 "LM358" H 4691 4305 50  0000 L CNN
-F 2 "" H 4350 4350 50  0001 C CNN
+F 2 "Housings_SOIC:SOIC-8_3.9x4.9mm_Pitch1.27mm" H 4350 4350 50  0001 C CNN
 F 3 "http://www.ti.com/lit/ds/symlink/lm2904-n.pdf" H 4350 4350 50  0001 C CNN
 	1    4350 4350
@@
 F 0 "U1" H 6641 4146 50  0000 L CNN
 F 1 "LM358" H 6641 4055 50  0000 L CNN
-F 2 "" H 6300 4100 50  0001 C CNN
+F 2 "Housings_SOIC:SOIC-8_3.9x4.9mm_Pitch1.27mm" H 6300 4100 50  0001 C CNN
 F 3 "http://www.ti.com/lit/ds/symlink/lm2904-n.pdf" H 6300 4100 50  0001 C CNN
 	2    6300 4100
@@
 F 0 "R4" H 3820 3696 50  0000 L CNN
 F 1 "10k" H 3820 3605 50  0000 L CNN
-F 2 "" V 3680 3650 50  0001 C CNN
+F 2 "Resistors_SMD:R_0402" V 3680 3650 50  0001 C CNN
 F 3 "" H 3750 3650 50  0001 C CNN
 	1    3750 3650
@@
 F 0 "R5" H 3820 4896 50  0000 L CNN
 F 1 "10k" H 3820 4805 50  0000 L CNN
-F 2 "" V 3680 4850 50  0001 C CNN
+F 2 "Resistors_SMD:R_0402" V 3680 4850 50  0001 C CNN
 F 3 "" H 3750 4850 50  0001 C CNN
 	1    3750 4850
@@
 F 0 "R2" V 3043 4450 50  0000 C CNN
 F 1 "1k" V 3134 4450 50  0000 C CNN
-F 2 "" V 3180 4450 50  0001 C CNN
+F 2 "Resistors_SMD:R_0402" V 3180 4450 50  0001 C CNN
 F 3 "" H 3250 4450 50  0001 C CNN
 	1    3250 4450
@@
 F 0 "R8" V 4393 5100 50  0000 C CNN
 F 1 "100k" V 4484 5100 50  0000 C CNN
-F 2 "" V 4530 5100 50  0001 C CNN
+F 2 "Resistors_SMD:R_0402" V 4530 5100 50  0001 C CNN
 F 3 "" H 4600 5100 50  0001 C CNN
 	1    4600 5100
@@
 F 0 "RV1" V 5586 4350 50  0000 C CNN
 F 1 "100k" V 5495 4350 50  0000 C CNN
-F 2 "" H 5700 4350 50  0001 C CNN
+F 2 "PCB-Condenser-Microphone:TC33X" H 5700 4350 50  0001 C CNN
 F 3 "" H 5700 4350 50  0001 C CNN
 	1    5700 4350
@@
 F 0 "R6" H 5520 3596 50  0000 L CNN
 F 1 "10k" H 5520 3505 50  0000 L CNN
-F 2 "" V 5380 3550 50  0001 C CNN
+F 2 "Resistors_SMD:R_0402" V 5380 3550 50  0001 C CNN
 F 3 "" H 5450 3550 50  0001 C CNN
 	1    5450 3550
@@
 F 0 "R7" H 5520 4896 50  0000 L CNN
 F 1 "10k" H 5520 4805 50  0000 L CNN
-F 2 "" V 5380 4850 50  0001 C CNN
+F 2 "Resistors_SMD:R_0402" V 5380 4850 50  0001 C CNN
 F 3 "" H 5450 4850 50  0001 C CNN
 	1    5450 4850
@@
 F 0 "C1" V 6098 3650 50  0000 C CNN
 F 1 "0.47uF" V 6189 3650 50  0000 C CNN
-F 2 "" H 6388 3500 50  0001 C CNN
+F 2 "Capacitors_SMD:C_0603_HandSoldering" H 6388 3500 50  0001 C CNN
 F 3 "" H 6350 3650 50  0001 C CNN
 	1    6350 3650
@@
 F 0 "J2" H 8212 4127 50  0000 R CNN
 F 1 "SJ-3523-SMT" H 8212 4218 50  0000 R CNN
-F 2 "" H 8700 4200 50  0001 C CNN
+F 2 "PCB-Condenser-Microphone:SJ-3523-SMT-TR" H 8700 4200 50  0001 C CNN
 F 3 "" H 8700 4200 50  0001 C CNN
 	1    8700 4200
@@
 Wire Wire Line
 	6500 3750 6500 3650
+$Comp
+L Mechanical:Mounting_Hole MT1
+U 1 1 5AA91E10
+P 950 1350
+F 0 "MT1" H 1050 1396 50  0000 L CNN
+F 1 "Strain Relief" H 1050 1305 50  0000 L CNN
+F 2 "Mounting_Holes:MountingHole_2.2mm_M2" H 950 1350 50  0001 C CNN
+F 3 "" H 950 1350 50  0001 C CNN
+	1    950  1350
+	1    0    0    -1
+$EndComp
+$Comp
+L Mechanical:Mounting_Hole MT2
+U 1 1 5AA9207A
+P 950 1550
+F 0 "MT2" H 1050 1596 50  0000 L CNN
+F 1 "Strain Relief" H 1050 1505 50  0000 L CNN
+F 2 "Mounting_Holes:MountingHole_2.2mm_M2" H 950 1550 50  0001 C CNN
+F 3 "" H 950 1550 50  0001 C CNN
+	1    950  1550
+	1    0    0    -1
+$EndComp
 $EndSCHEMATC

Commit message: Layd out pcb and added OSHW logo
Parts:
- J1: footprint Pin_Headers:Pin_Header_Angled_1x02_Pitch2.54mm -> Pin_Headers:Pin_Header_Straight_1x02_Pitch2.54mm
Changed lines of the file:
@@
 F 0 "J1" H 1900 1200 50  0000 C CNN
 F 1 "Conn_01x02" H 1900 1300 50  0000 C CNN
-F 2 "Pin_Headers:Pin_Header_Angled_1x02_Pitch2.54mm" H 1750 1500 50  0001 C CNN
+F 2 "Pin_Headers:Pin_Header_Straight_1x02_Pitch2.54mm" H 1750 1500 50  0001 C CNN
 F 3 "~" H 1750 1500 50  0001 C CNN
 	1    1750 1500

Commit message: Updated schimatic to have fet preamp
Parts:
- added C5: 680pF, Capacitors_SMD:C_0805_HandSoldering, symbol device:C
- added Q1: Q_NJFET_DSG, symbol device:Q_NJFET_DSG
- added R11: 100M, Resistors_SMD:R_0402, symbol device:R
- added R3: 1k, Resistors_SMD:R_0402, symbol device:R
- added R4: 10k, Resistors_SMD:R_0402, symbol device:R
- R10: renamed from R3; value 10k -> 100M
- renumbered R4 to R5, R5 to R6, R6 to R7, R7 to R8, R8 to R9
Connections:
- wire segments 48 -> 57
Changed lines of the file:
@@
 L device:Microphone_Condenser MK1
 U 1 1 5AA49771
-P 2200 4800
-F 0 "MK1" H 2330 4846 50  0000 L CNN
-F 1 "Microphone_Condenser" H 2330 4755 50  0000 L CNN
-F 2 "PCB-Condenser-Microphone:Condenser-Microphone-Backplate-30mm-Single-mount" V 2200 4900 50  0001 C CNN
-F 3 "" V 2200 4900 50  0001 C CNN
-	1    2200 4800
+P 1050 5250
+F 0 "MK1" H 1180 5296 50  0000 L CNN
+F 1 "Microphone_Condenser" H 1180 5205 50  0000 L CNN
+F 2 "PCB-Condenser-Microphone:Condenser-Microphone-Backplate-30mm-Single-mount" V 1050 5350 50  0001 C CNN
+F 3 "" V 1050 5350 50  0001 C CNN
+	1    1050 5250
 	1    0    0    -1
 $EndComp
@@
 L power:GND #PWR0102
 U 1 1 5AA4992F
-P 2200 5100
-F 0 "#PWR0102" H 2200 4850 50  0001 C CNN
-F 1 "GND" H 2205 4927 50  0000 C CNN
-F 2 "" H 2200 5100 50  0001 C CNN
-F 3 "" H 2200 5100 50  0001 C CNN
-	1    2200 5100
-	1    0    0    -1
-$EndComp
-Wire Wire Line
-	2200 5100 2200 5000
+P 1050 5550
+F 0 "#PWR0102" H 1050 5300 50  0001 C CNN
+F 1 "GND" H 1055 5377 50  0000 C CNN
+F 2 "" H 1050 5550 50  0001 C CNN
+F 3 "" H 1050 5550 50  0001 C CNN
+	1    1050 5550
+	1    0    0    -1
+$EndComp
+Wire Wire Line
+	1050 5550 1050 5450
 $Comp
 L Connector:Conn_01x02 J1
@@
 L power:+9V #PWR0106
 U 1 1 5AA79FC3
-P 2200 3900
-F 0 "#PWR0106" H 2200 3750 50  0001 C CNN
-F 1 "+9V" H 2215 4073 50  0000 C CNN
-F 2 "" H 2200 3900 50  0001 C CNN
-F 3 "" H 2200 3900 50  0001 C CNN
-	1    2200 3900
-	1    0    0    -1
-$EndComp
-$Comp
-L device:R R3
+P 1050 4350
+F 0 "#PWR0106" H 1050 4200 50  0001 C CNN
+F 1 "+9V" H 1065 4523 50  0000 C CNN
+F 2 "" H 1050 4350 50  0001 C CNN
+F 3 "" H 1050 4350 50  0001 C CNN
+	1    1050 4350
+	1    0    0    -1
+$EndComp
+$Comp
+L device:R R10
 U 1 1 5AA7A003
-P 2200 4150
-F 0 "R3" H 2270 4196 50  0000 L CNN
-F 1 "10k" H 2270 4105 50  0000 L CNN
-F 2 "Resistors_SMD:R_0402" V 2130 4150 50  0001 C CNN
-F 3 "" H 2200 4150 50  0001 C CNN
-	1    2200 4150
-	1    0    0    -1
-$EndComp
-Wire Wire Line
-	2200 4000 2200 3900
-Wire Wire Line
-	2200 4600 2200 4450
+P 1050 4600
+F 0 "R10" H 1120 4646 50  0000 L CNN
+F 1 "100M" H 1120 4555 50  0000 L CNN
+F 2 "Resistors_SMD:R_0402" V 980 4600 50  0001 C CNN
+F 3 "" H 1050 4600 50  0001 C CNN
+	1    1050 4600
+	1    0    0    -1
+$EndComp
+Wire Wire Line
+	1050 4450 1050 4350
+Wire Wire Line
+	1050 5050 1050 4900
 $Comp
 L device:C C3
@@
 $EndComp
 Wire Wire Line
-	2200 4450 2600 4450
-Connection ~ 2200 4450
-Wire Wire Line
-	2200 4450 2200 4300
+	1050 4900 1450 4900
+Connection ~ 1050 4900
+Wire Wire Line
+	1050 4900 1050 4750
 $Comp
 L device:C C4
@@
 	6200 4500 6200 4400
 $Comp
-L device:R R4
+L device:R R5
 U 1 1 5AA83723
 P 3750 3650
-F 0 "R4" H 3820 3696 50  0000 L CNN
+F 0 "R5" H 3820 3696 50  0000 L CNN
 F 1 "10k" H 3820 3605 50  0000 L CNN
 F 2 "Resistors_SMD:R_0402" V 3680 3650 50  0001 C CNN
@@
 $EndComp
 $Comp
-L device:R R5
+L device:R R6
 U 1 1 5AA837B4
 P 3750 4850
-F 0 "R5" H 3820 4896 50  0000 L CNN
+F 0 "R6" H 3820 4896 50  0000 L CNN
 F 1 "10k" H 3820 4805 50  0000 L CNN
 F 2 "Resistors_SMD:R_0402" V 3680 4850 50  0001 C CNN
@@
 	3750 3500 3750 3350
 $Comp
-L device:R R8
+L device:R R9
 U 1 1 5AA852B6
 P 4600 5100
-F 0 "R8" V 4393 5100 50  0000 C CNN
+F 0 "R9" V 4393 5100 50  0000 C CNN
 F 1 "100k" V 4484 5100 50  0000 C CNN
 F 2 "Resistors_SMD:R_0402" V 4530 5100 50  0001 C CNN
@@
 	6900 4100 7800 4100
 $Comp
-L device:R R6
+L device:R R7
 U 1 1 5AA88985
 P 5450 3550
-F 0 "R6" H 5520 3596 50  0000 L CNN
+F 0 "R7" H 5520 3596 50  0000 L CNN
 F 1 "10k" H 5520 3505 50  0000 L CNN
 F 2 "Resistors_SMD:R_0402" V 5380 3550 50  0001 C CNN
@@
 $EndComp
 $Comp
-L device:R R7
+L device:R R8
 U 1 1 5AA889D7
 P 5450 4850
-F 0 "R7" H 5520 4896 50  0000 L CNN
+F 0 "R8" H 5520 4896 50  0000 L CNN
 F 1 "10k" H 5520 4805 50  0000 L CNN
 F 2 "Resistors_SMD:R_0402" V 5380 4850 50  0001 C CNN
@@
 	1    0    0    -1
 $EndComp
+$Comp
+L device:C C5
+U 1 1 5AB86155
+P 1600 4900
+F 0 "C5" V 1348 4900 50  0000 C CNN
+F 1 "680pF" V 1439 4900 50  0000 C CNN
+F 2 "Capacitors_SMD:C_0805_HandSoldering" H 1638 4750 50  0001 C CNN
+F 3 "" H 1600 4900 50  0001 C CNN
+	1    1600 4900
+	0    1    1    0
+$EndComp
+$Comp
+L device:Q_NJFET_DSG Q1
+U 1 1 5AB877EE
+P 2500 4900
+F 0 "Q1" H 2691 4946 50  0000 L CNN
+F 1 "Q_NJFET_DSG" H 2691 4855 50  0000 L CNN
+F 2 "" H 2700 5000 50  0001 C CNN
+F 3 "" H 2500 4900 50  0001 C CNN
+	1    2500 4900
+	1    0    0    -1
+$EndComp
+$Comp
+L device:R R11
+U 1 1 5AB8812B
+P 2100 5200
+F 0 "R11" H 2170 5246 50  0000 L CNN
+F 1 "100M" H 2170 5155 50  0000 L CNN
+F 2 "Resistors_SMD:R_0402" V 2030 5200 50  0001 C CNN
+F 3 "" H 2100 5200 50  0001 C CNN
+	1    2100 5200
+	1    0    0    -1
+$EndComp
+$Comp
+L power:GND #PWR?
+U 1 1 5AB881B7
+P 2100 5550
+F 0 "#PWR?" H 2100 5300 50  0001 C CNN
+F 1 "GND" H 2105 5377 50  0000 C CNN
+F 2 "" H 2100 5550 50  0001 C CNN
+F 3 "" H 2100 5550 50  0001 C CNN
+	1    2100 5550
+	1    0    0    -1
+$EndComp
+Wire Wire Line
+	2100 5550 2100 5350
+Wire Wire Line
+	2100 5050 2100 4900
+Wire Wire Line
+	2100 4900 2300 4900
+Wire Wire Line
+	1750 4900 2100 4900
+Connection ~ 2100 4900
+$Comp
+L device:R R4
+U 1 1 5AB8CE07
+P 2600 3900
+F 0 "R4" H 2670 3946 50  0000 L CNN
+F 1 "10k" H 2670 3855 50  0000 L CNN
+F 2 "Resistors_SMD:R_0402" V 2530 3900 50  0001 C CNN
+F 3 "" H 2600 3900 50  0001 C CNN
+	1    2600 3900
+	1    0    0    -1
+$EndComp
+Wire Wire Line
+	2600 4700 2600 4450
+Connection ~ 2600 4450
+Wire Wire Line
+	2600 4450 2600 4050
+$Comp
+L power:+9V #PWR?
+U 1 1 5AB8EBFE
+P 2600 3350
+F 0 "#PWR?" H 2600 3200 50  0001 C CNN
+F 1 "+9V" H 2615 3523 50  0000 C CNN
+F 2 "" H 2600 3350 50  0001 C CNN
+F 3 "" H 2600 3350 50  0001 C CNN
+	1    2600 3350
+	1    0    0    -1
+$EndComp
+Wire Wire Line
+	2600 3750 2600 3350
+$Comp
+L device:R R3
+U 1 1 5AB8F94F
+P 2600 5350
+F 0 "R3" H 2670 5396 50  0000 L CNN
+F 1 "1k" H 2670 5305 50  0000 L CNN
+F 2 "Resistors_SMD:R_0402" V 2530 5350 50  0001 C CNN
+F 3 "" H 2600 5350 50  0001 C CNN
+	1    2600 5350
+	1    0    0    -1
+$EndComp
+Wire Wire Line
+	2600 5200 2600 5100
+$Comp
+L power:GND #PWR?
+U 1 1 5AB90746
+P 2600 5600
+F 0 "#PWR?" H 2600 5350 50  0001 C CNN
+F 1 "GND" H 2605 5427 50  0000 C CNN
+F 2 "" H 2600 5600 50  0001 C CNN
+F 3 "" H 2600 5600 50  0001 C CNN
+	1    2600 5600
+	1    0    0    -1
+$EndComp
+Wire Wire Line
+	2600 5600 2600 5500
 $EndSCHEMATC

Commit message: Updated circuit to match the jfet
Parts:
- removed R3: 1k, Resistors_SMD:R_0402, symbol device:R
- C5: footprint Capacitors_SMD:C_0805_HandSoldering -> Capacitors_SMD:C_0603_HandSoldering
- Q1: footprint (none) -> TO_SOT_Packages_SMD:SOT-23_Handsoldering
- R3: renamed from R4; value 10k -> 300
- renumbered R11 to R10, R5 to R4, R6 to R5, R7 to R6, R8 to R7, R9 to R8, R10 to R9
Connections:
- wire segments 57 -> 56
Changed lines of the file:
@@
 $EndComp
 $Comp
-L device:R R10
+L device:R R9
 U 1 1 5AA7A003
 P 1050 4600
-F 0 "R10" H 1120 4646 50  0000 L CNN
+F 0 "R9" H 1120 4646 50  0000 L CNN
 F 1 "100M" H 1120 4555 50  0000 L CNN
 F 2 "Resistors_SMD:R_0402" V 980 4600 50  0001 C CNN
@@
 	6200 4500 6200 4400
 $Comp
-L device:R R5
+L device:R R4
 U 1 1 5AA83723
 P 3750 3650
-F 0 "R5" H 3820 3696 50  0000 L CNN
+F 0 "R4" H 3820 3696 50  0000 L CNN
 F 1 "10k" H 3820 3605 50  0000 L CNN
 F 2 "Resistors_SMD:R_0402" V 3680 3650 50  0001 C CNN
@@
 $EndComp
 $Comp
-L device:R R6
+L device:R R5
 U 1 1 5AA837B4
 P 3750 4850
-F 0 "R6" H 3820 4896 50  0000 L CNN
+F 0 "R5" H 3820 4896 50  0000 L CNN
 F 1 "10k" H 3820 4805 50  0000 L CNN
 F 2 "Resistors_SMD:R_0402" V 3680 4850 50  0001 C CNN
@@
 	3750 3500 3750 3350
 $Comp
-L device:R R9
+L device:R R8
 U 1 1 5AA852B6
 P 4600 5100
-F 0 "R9" V 4393 5100 50  0000 C CNN
+F 0 "R8" V 4393 5100 50  0000 C CNN
 F 1 "100k" V 4484 5100 50  0000 C CNN
 F 2 "Resistors_SMD:R_0402" V 4530 5100 50  0001 C CNN
@@
 	6900 4100 7800 4100
 $Comp
-L device:R R7
+L device:R R6
 U 1 1 5AA88985
 P 5450 3550
-F 0 "R7" H 5520 3596 50  0000 L CNN
+F 0 "R6" H 5520 3596 50  0000 L CNN
 F 1 "10k" H 5520 3505 50  0000 L CNN
 F 2 "Resistors_SMD:R_0402" V 5380 3550 50  0001 C CNN
@@
 $EndComp
 $Comp
-L device:R R8
+L device:R R7
 U 1 1 5AA889D7
 P 5450 4850
-F 0 "R8" H 5520 4896 50  0000 L CNN
+F 0 "R7" H 5520 4896 50  0000 L CNN
 F 1 "10k" H 5520 4805 50  0000 L CNN
 F 2 "Resistors_SMD:R_0402" V 5380 4850 50  0001 C CNN
@@
 F 0 "C5" V 1348 4900 50  0000 C CNN
 F 1 "680pF" V 1439 4900 50  0000 C CNN
-F 2 "Capacitors_SMD:C_0805_HandSoldering" H 1638 4750 50  0001 C CNN
+F 2 "Capacitors_SMD:C_0603_HandSoldering" H 1638 4750 50  0001 C CNN
 F 3 "" H 1600 4900 50  0001 C CNN
 	1    1600 4900
@@
 F 0 "Q1" H 2691 4946 50  0000 L CNN
 F 1 "Q_NJFET_DSG" H 2691 4855 50  0000 L CNN
-F 2 "" H 2700 5000 50  0001 C CNN
+F 2 "TO_SOT_Packages_SMD:SOT-23_Handsoldering" H 2700 5000 50  0001 C CNN
 F 3 "" H 2500 4900 50  0001 C CNN
 	1    2500 4900
@@
 $EndComp
 $Comp
-L device:R R11
+L device:R R10
 U 1 1 5AB8812B
 P 2100 5200
-F 0 "R11" H 2170 5246 50  0000 L CNN
+F 0 "R10" H 2170 5246 50  0000 L CNN
 F 1 "100M" H 2170 5155 50  0000 L CNN
 F 2 "Resistors_SMD:R_0402" V 2030 5200 50  0001 C CNN
@@
 $EndComp
 $Comp
-L power:GND #PWR?
+L power:GND #PWR0118
 U 1 1 5AB881B7
 P 2100 5550
-F 0 "#PWR?" H 2100 5300 50  0001 C CNN
+F 0 "#PWR0118" H 2100 5300 50  0001 C CNN
 F 1 "GND" H 2105 5377 50  0000 C CNN
 F 2 "" H 2100 5550 50  0001 C CNN
@@
 Connection ~ 2100 4900
 $Comp
-L device:R R4
+L device:R R3
 U 1 1 5AB8CE07
 P 2600 3900
-F 0 "R4" H 2670 3946 50  0000 L CNN
-F 1 "10k" H 2670 3855 50  0000 L CNN
+F 0 "R3" H 2670 3946 50  0000 L CNN
+F 1 "300" H 2670 3855 50  0000 L CNN
 F 2 "Resistors_SMD:R_0402" V 2530 3900 50  0001 C CNN
 F 3 "" H 2600 3900 50  0001 C CNN
@@
 	2600 4450 2600 4050
 $Comp
-L power:+9V #PWR?
+L power:+9V #PWR0119
 U 1 1 5AB8EBFE
 P 2600 3350
-F 0 "#PWR?" H 2600 3200 50  0001 C CNN
+F 0 "#PWR0119" H 2600 3200 50  0001 C CNN
 F 1 "+9V" H 2615 3523 50  0000 C CNN
 F 2 "" H 2600 3350 50  0001 C CNN
@@
 	2600 3750 2600 3350
 $Comp
-L device:R R3
-U 1 1 5AB8F94F
-P 2600 5350
-F 0 "R3" H 2670 5396 50  0000 L CNN
-F 1 "1k" H 2670 5305 50  0000 L CNN
-F 2 "Resistors_SMD:R_0402" V 2530 5350 50  0001 C CNN
-F 3 "" H 2600 5350 50  0001 C CNN
-	1    2600 5350
-	1    0    0    -1
-$EndComp
-Wire Wire Line
-	2600 5200 2600 5100
-$Comp
-L power:GND #PWR?
+L power:GND #PWR0120
 U 1 1 5AB90746
 P 2600 5600
-F 0 "#PWR?" H 2600 5350 50  0001 C CNN
+F 0 "#PWR0120" H 2600 5350 50  0001 C CNN
 F 1 "GND" H 2605 5427 50  0000 C CNN
 F 2 "" H 2600 5600 50  0001 C CNN
@@
 $EndComp
 Wire Wire Line
-	2600 5600 2600 5500
+	2600 5600 2600 5100
 $EndSCHEMATC

Commit message: Uodated JFET
Parts:
- R3: value 300 -> 10K
Changed lines of the file:
@@
 P 2600 3900
 F 0 "R3" H 2670 3946 50  0000 L CNN
-F 1 "300" H 2670 3855 50  0000 L CNN
+F 1 "10K" H 2670 3855 50  0000 L CNN
 F 2 "Resistors_SMD:R_0402" V 2530 3900 50  0001 C CNN
 F 3 "" H 2600 3900 50  0001 C CNN
