File: PCB-Condenser-Microphone/PCB-Condenser-Microphone.sch (KiCad schematic (older format))
At the start: 25 parts, among them J1 Conn_01x02, J2 SJ-3523-SMT, Q1 Q_NJFET_DSG, SW1 SW_SPDT, U1 LM358

Commit message: Updated files for new library
Parts:
- C1, C2, C3, C4, C5: symbol device:C -> Device:C
- D1: symbol device:LED -> Device:LED
- J1: symbol Connector:Conn_01x02 -> Connector_Generic:Conn_01x02
- MK1: symbol device:Microphone_Condenser -> Device:Microphone_Condenser
- Q1: symbol device:Q_NJFET_DSG -> Device:Q_NJFET_DSG
- R1, R10, R2, R3, R4, R5, R6, R7, R8, R9: symbol device:R -> Device:R
- RV1: symbol device:POT -> Device:POT
- U1: symbol linear:LM358 -> Amplifier_Operational:LM358
Changed lines of the file:
@@
 	9100 3900 9100 4000
 $Comp
-L device:Microphone_Condenser MK1
+L Device:Microphone_Condenser MK1
 U 1 1 5AA49771
 P 1050 5250
@@
 	1050 5550 1050 5450
 $Comp
-L Connector:Conn_01x02 J1
+L Connector_Generic:Conn_01x02 J1
 U 1 1 5AA797B8
 P 1750 1500
@@
 $EndComp
 $Comp
-L device:R R9
+L Device:R R9
 U 1 1 5AA7A003
 P 1050 4600
@@
 	1050 5050 1050 4900
 $Comp
-L device:C C3
+L Device:C C3
 U 1 1 5AA7A11B
 P 2750 4450
@@
 	1050 4900 1050 4750
 $Comp
-L device:C C4
+L Device:C C4
 U 1 1 5AA7A7A1
 P 7950 4100
@@
 	8100 4100 8350 4100
 $Comp
-L device:C C2
+L Device:C C2
 U 1 1 5AA7A941
 P 2850 1450
@@
 	2600 1600 2850 1600
 $Comp
-L device:LED D1
+L Device:LED D1
 U 1 1 5AA7AE30
 P 3700 1900
@@
 	3700 1750 3700 1650
 $Comp
-L device:R R1
+L Device:R R1
 U 1 1 5AA7B2D1
 P 3700 2300
@@
 Connection ~ 2600 1600
 $Comp
-L linear:LM358 U1
+L Amplifier_Operational:LM358 U1
 U 1 1 5AA829BD
 P 4350 4350
@@
 $EndComp
 $Comp
-L linear:LM358 U1
+L Amplifier_Operational:LM358 U1
 U 2 1 5AA82BBE
 P 6300 4100
@@
 	6200 4500 6200 4400
 $Comp
-L device:R R4
+L Device:R R4
 U 1 1 5AA83723
 P 3750 3650
@@
 $EndComp
 $Comp
-L device:R R5
+L Device:R R5
 U 1 1 5AA837B4
 P 3750 4850
@@
 $EndComp
 $Comp
-L device:R R2
+L Device:R R2
 U 1 1 5AA8402D
 P 3250 4450
@@
 	3750 3500 3750 3350
 $Comp
-L device:R R8
+L Device:R R8
 U 1 1 5AA852B6
 P 4600 5100
@@
 	4000 4450 4050 4450
 $Comp
-L device:POT RV1
+L Device:POT RV1
 U 1 1 5AA8621E
 P 5700 4350
@@
 	6900 4100 7800 4100
 $Comp
-L device:R R6
+L Device:R R6
 U 1 1 5AA88985
 P 5450 3550
@@
 $EndComp
 $Comp
-L device:R R7
+L Device:R R7
 U 1 1 5AA889D7
 P 5450 4850
@@
 	5450 4000 5450 4700
 $Comp
-L device:C C1
+L Device:C C1
 U 1 1 5AA8CA57
 P 6350 3650
@@
 $EndComp
 $Comp
-L device:C C5
+L Device:C C5
 U 1 1 5AB86155
 P 1600 4900
@@
 $EndComp
 $Comp
-L device:Q_NJFET_DSG Q1
+L Device:Q_NJFET_DSG Q1
 U 1 1 5AB877EE
 P 2500 4900
@@
 $EndComp
 $Comp
-L device:R R10
+L Device:R R10
 U 1 1 5AB8812B
 P 2100 5200
@@
 Connection ~ 2100 4900
 $Comp
-L device:R R3
+L Device:R R3
 U 1 1 5AB8CE07
 P 2600 3900
