File: PCB-Condenser-Microphone-Backplate/PCB-Condenser-Microphone-Backplate.sch (KiCad schematic (older format))
At the start: 1 part

Commit message: Updated files for new library
Parts:
- MK1: symbol device:Microphone_Condenser -> Device:Microphone_Condenser
Changed lines of the file:
@@
 $EndDescr
 $Comp
-L device:Microphone_Condenser MK1
+L Device:Microphone_Condenser MK1
 U 1 1 5AA49771
 P 2350 2950
